Commit message: Add files via upload

File: src/goalkeeper_description/urdf/goalkeeper.urdf (robot description, URDF)
Before this commit: robot goalkeeper_robot, 5 links, 4 joints
Links:
- removed link defense_plate
- removed link vertical_extension
- added link keeper_body, mass 85; collision box size=0.24 0.12 0.1; collision box size=0.24 0.15 0.22
- link base_link: mass 1.0 -> 0.001; geometry 
- link slider_carriage: mass 0.5 -> 0.001; geometry 
Joints:
- removed joint plate_fixed_joint
- removed joint slider_joint
- removed joint vertical_joint
- added joint slide_joint: type prismatic, parent base_link, child slider_carriage, origin xyz=0 0 0 rpy=0 0 0, axis 0 1 0, limit lower=-3.2 upper=3.2 effort=2000 velocity=2
- added joint tilt_joint: type revolute, parent slider_carriage, child keeper_body, origin xyz=0 0 1 rpy=0 0 0, axis 1 0 0, limit lower=-0.7853981633974483 upper=0.7853981633974483 effort=2000 velocity=4
- joint world_to_base: origin xyz=0 0 0 rpy=0 0 0 -> (none)
